File: CoralWave.kicad_sch (KiCad schematic)
At the start: 45 parts, among them IC1 ESP32-C3-WROOM-02-N4, IC2 TLV62568DBVR, J1 73251-1290, J2 USB4105-GF-A, U1 CC1101RGP, Y1 NX3225GA-26MHZ

Commit message: Add BOM
Other:
- company: CodingCorals -> mineiwik
Changed lines of the file:
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@@
   (title_block
     (title "CoralWave")
-    (date "2023-07-16")
+    (date "2023-08-22")
     (rev "1.0")
-    (company "CodingCorals")
+    (company "mineiwik")
   )
   (junction (at 38.1 144.78) (diameter 0) (color 0 0 0 0)
